Commit message: ur_automata_hsi: hyperspectral measurement after the 3D scan
hsi_node waits for an object on /hsi/start (MQTT automata/hsi/start). From
home only, it moves the HSI frame (ee_automata_hsi, new URDF link: tool0 +
(0, 0.072, 0.091), 83.5 mm closer to the flange and 20 mm further forward
than the camera) 0.30 m above the scan center, looking down, with the
rotation about the vertical whose IK is closest to home; sends the request
on /hsi/acquire (hsi/commands), waits for measure_complete on /hsi/status
(hsi/status), goes back home and reports /hsi/done (automata/hsi/done).

- one MQTT bridge for the cell: mqtt_bridge.launch.py in ur_automata_bringup,
  included by the one-command launcher (no longer in scan_tsp.launch.py)
- launcher: use_hsi (default true); speed (default 0.4) is the same for the
  scan and the HSI motions
- docs: HSI topics and the message contract for the HSI app

File: src/automata_robot/ur_automata_description/urdf/ur_automata.urdf.xacro (robot description, xacro)
@@ -121,3 +121,13 @@
   </joint>
   <link name="ee_automata_tcp"/>
+  <!-- Hyperspectral sensor (HSI) on the same end effector: 83.5 mm closer to
+       the flange than the camera (z 174.5 - 83.5 = 91 mm) and 20 mm further
+       forward, toward the object (y 52 + 20 = 72 mm). It looks along Y, like
+       the camera. Used by ur_automata_hsi. -->
+  <joint name="ee_automata_hsi_fixed_joint" type="fixed">
+    <origin xyz="0 0.072 0.091" rpy="0 0 0"/>
+    <parent link="tool0"/>
+    <child link="ee_automata_hsi"/>
+  </joint>
+  <link name="ee_automata_hsi"/>
 </robot>
